File: circuit/LIS3MDLTR/LIS3MDLTR/LIS3MDLTR.kicad_sch (KiCad schematic)
At the start: 9 parts, among them U1 LIS3MDLTR, U2 LIS3MDLTR, U3 LIS3MDLTR, U4 LIS3MDLTR

Commit message: idk
Parts:
- removed U1, U2, U3, U4: LIS3MDLTR, LIS3MDL:LIS3MDLTR, symbol LIS3MDL Magnetometer:LIS3MDLTR
- added C4: 0.1uF, symbol Device:C
- added C5: 1uF, symbol Device:C
- added R3, R4: R, symbol Device:R
- added U1: AP2112K-3.3TRG1, SOT_RG1_DIO, symbol AP2112K-3.3TRG1:AP2112K-3.3TRG1
- C1: value 100nF -> 0.1uF; footprint Capacitor_SMD:C_0201_0603Metric -> (none)
- C2: value 1uF -> 10uF; footprint Capacitor_SMD:C_0201_0603Metric -> (none); Comment Electrolytic -> (none)
- C3: value 100nF -> 10uF; footprint Capacitor_SMD:C_0201_0603Metric -> (none); Comment Ceramic,close to Vdd -> (none)
- R1, R2: footprint Resistor_SMD:R_0201_0603Metric -> (none)
Connections:
- net GND: now also C2.2, C3.2, C4.2, C5.2, U1.2 (GND); no longer C2.1, C3.1
- net +3V3: now reaches C1.1
- net +3V3: now also C3.1, C5.1, U1.5 (VOUT)
- removed net +2V5: C2.2, C3.2, R1.1, R2.1
- net SDI: no longer names the net of R1.2
- net SDO: no longer names the net of R2.2
- new net CAP: C4.1
- new net VCC: C2.1, U1.1 (VIN), U1.3 (EN)
- no-connect marks 1 -> 0

Commit message: Finished LIS3MDL schematic
Parts:
- added D1, D2, D3, D4: 1N4148, Diode_THT:D_DO-35_SOD27_P7.62mm_Horizontal, symbol Diode:1N4148
- added Q1, Q2: BSS138, Package_TO_SOT_SMD:SOT-23, symbol Transistor_FET:BSS138
- added R5, R6, R7, R8, R9: 10k, symbol Device:R
- added U2, U3, U4, U5: LIS3MDLTR, LGA-12_2X2X1_STM, symbol LIS3MDL Magnetometer:LIS3MDLTR
- R3, R4: value R -> 10k
- renumbered C2 to C1, C3 to C2, C5 to C3, C1 to C4, C4 to C5
Connections:
- net +3V3: now also R3.1, R4.1, Q1.1 (G), Q2.1 (G), R5.2, R6.1, R7.1, R8.1, U2.5 (VDD), U2.6 (VDD_IO), U3.5 (VDD), U3.6 (VDD_IO), U4.5 (VDD), U4.6 (VDD_IO), U5.5 (VDD), U5.6 (VDD_IO)
- net CAP: now also U2.4 (C1), U3.4 (C1), U4.4 (C1), U5.4 (C1)
- net GND: now also R9.1, U2.3 (GND), U3.3 (GND), U4.3 (GND), U5.3 (GND)
- net VCC: now also R1.1, R2.1
- net SPC: now reaches R1.2
- net SPC: now also R3.2, Q1.2 (S), Q1.3 (D), U2.1 (SCL/SPC), U3.1 (SCL/SPC), U4.1 (SCL/SPC), U5.1 (SCL/SPC)
- net SDI_3V: now reaches R4.2
- net SDI_3V: now also Q2.2 (S), U2.11 (SDA/SDI/SDO), U3.11 (SDA/SDI/SDO), U4.11 (SDA/SDI/SDO), U5.11 (SDA/SDI/SDO)
- net SDI: now reaches R2.2
- net SDI: now also Q2.3 (D)
- new net CS1: D4.2 (A), R5.1, U2.10 (CS)
- new net CS1_5V: D4.1 (K)
- new net CS2: D1.2 (A), R6.2, U4.10 (CS)
- new net CS2_5V: D1.1 (K)
- new net CS3: D2.2 (A), R7.2, U3.10 (CS)
- new net CS3_5V: D2.1 (K)
- new net CS4: D3.2 (A), R8.2, U5.10 (CS)
- new net CS4_5V: D3.1 (K)
- new net DRDY1: U2.8 (DRDY)
- new net DRDY2: U4.8 (DRDY)
- new net DRDY3: U3.8 (DRDY)
- new net DRDY4: U5.8 (DRDY)
- new net INT1: U2.7 (INT)
- new net INT2: U4.7 (INT)
- new net INT3: U3.7 (INT)
- new net INT4: U5.7 (INT)
- new net SDO: R9.2, U2.9 (SDO/SA1), U3.9 (SDO/SA1), U4.9 (SDO/SA1), U5.9 (SDO/SA1)
